File: sch/tow/tow.kicad_pcb (KiCad board)
At the start: 2 copper layers, 160 x 40.6 mm, 32 parts, among them J1 Conn_02x01, U1 R-78E5.0-1.0, U2 ATMEGA328P_PDIP, Y1 16MHZ

Commit message: Updated PCB
Parts:
- removed R3, R4: 1k, Resistor_THT:R_Axial_DIN0207_L6.3mm_D2.5mm_P10.16mm_Horizontal
- Y1: value 16MHZ -> CRYSTAL-16MHZPTH-HC49US
Routing:
- net /5v: track 135.6 -> 85.6 mm
- net Net-(S2-Pad3): track 69.5 -> 62.9 mm
- net Net-(S3-Pad3): track 80.0 -> 77.3 mm
